Commit message: interaction between state machine and action client

File: urdf/robot.xacro (robot description, xacro)
@@ -16,5 +16,5 @@
      	</geometry>
 	</xacro:macro>
-  <material name="black">
+    <material name="black">
     <color rgba="0.0 0.0 0.0 1.0"/>
   </material>
@@ -115,17 +115,69 @@
     <joint_properties damping="1.0" friction="1.0"/>
   </joint>
+<link name="neck_link">
+  	<inertial>
+  		<mass value="0.025"/>
+  		<origin xyz="0 0 0" rpy="0 0 0" />
+  		<inertia ixx="0.000010279" ixy="0" ixz="0" iyy="0.000010279" iyz="0" izz="0.000007225"/>
+  	</inertial>
+  	<collision>
+  	  <origin xyz="0 0 0.025" rpy="0 0 0"/>
+      <geometry>
+        <cylinder radius="0.04" length="0.05"/>
+      </geometry>
+  	</collision>
+  	<visual>
+  	  <origin xyz="0 0 0.025" rpy="0 0 0"/>
+      <geometry>
+        <cylinder radius="0.06" length="0.05"/>
+      </geometry>
+      <material name="orange" />
+  	</visual>
+  </link>
+ <joint name="neck_joint" type="fixed">
+  	<origin rpy="0 0 0" xyz="0.17 0 0.035"/>
+  	<parent link="link_chassis"/>
+  	<child link="neck_link"/>
+  </joint>
+ <link name="head_link">
+  	<inertial>
+  		<mass value="0.1"/>
+  		<origin xyz="0 0 0" rpy="0 0 0" />
+  		<inertia ixx="0.0000416666667" ixy="0" ixz="0" iyy="0.0000416666667" iyz="0" izz="0.0000416666667"/>
+  	</inertial>
+  	<collision>
+  	  <origin xyz="0 0 0.075" rpy="0 0 0"/>
+      <geometry>
+        <box size="0.15 0.15 0.15"/>
+      </geometry>
+  	</collision>
+  	<visual>
+  	  <origin xyz="0 0 0.075" rpy="0 0 0"/>
+      <geometry>
+        <box size="0.15 0.15 0.15"/>
+      </geometry>
+      <material name="green"/>
+  	</visual>
+  </link>
+  <joint name="head_joint" type="revolute">
+  	<axis xyz="0 0 1"/>
+  	<limit effort="1000.0" lower="-6.28" upper="6.28" velocity="0.2"/>
+  	<origin rpy="0 0 0" xyz="0 0 0.05"/>
+  	<parent link="neck_link"/>
+  	<child link="head_link"/>
+  </joint>
   <link name="camera_link">
 	    <collision>
 	      <origin xyz="0 0 0.025" rpy="0 0 0"/>
 	      <geometry>
-		<box size="0.05 0.05 0.05"/>
+		<box size="0.05 0.05 0.01"/>
 	      </geometry>
 	    </collision>
 	    <visual>
-	      <origin xyz="0 0 0.025" rpy="0 0 0"/>
+	      <origin xyz="0 0 0.005" rpy="0 0 0"/>
 	      <geometry>
-		<box size="0.05 0.05 0.05"/>
+		<box size="0.05 0.05 0.01"/>
 	      </geometry>
-	      <material name="red">
+	      <material name="blue">
 		<color rgba="1 0 0 1"/>
 	      </material>
@@ -133,5 +185,5 @@
 	    <inertial>
 	      <mass value="1e-5" />
-	      <origin xyz="0 0 0" rpy="0 0 0"/>
+	      <origin xyz="0 0 0.005" rpy="0 0 0"/>
 	      <inertia ixx="1e-6" ixy="0" ixz="0" iyy="1e-6" iyz="0" izz="1e-6" />
 	    </inertial>
@@ -139,6 +191,6 @@
   <joint name="camera_joint" type="fixed">
 	    <axis xyz="0 1 0" />
-	    <origin xyz="0.23 0 0.0" rpy="0 0 0"/>
-	    <parent link="link_chassis"/>
+	    <origin xyz="0.05 0 0.15" rpy="0 0 0"/>
+	    <parent link="head_link"/>
 	    <child link="camera_link"/>
 	 </joint>

Commit message: robot moving head

File: urdf/robot.xacro (robot description, xacro)
@@ -134,6 +134,8 @@
       <material name="orange" />
   	</visual>
-  </link>
- <joint name="neck_joint" type="fixed">
+</link>
+ <joint name="neck_joint" type="revolute">
+	<axis xyz="0 0 1"/>
+  	<limit effort="1000.0" lower="0" upper="6.28" velocity="0.2"/>
   	<origin rpy="0 0 0" xyz="0.17 0 0.035"/>
   	<parent link="link_chassis"/>
@@ -157,10 +159,7 @@
         <box size="0.15 0.15 0.15"/>
       </geometry>
-      <material name="green"/>
   	</visual>
   </link>
-  <joint name="head_joint" type="revolute">
-  	<axis xyz="0 0 1"/>
-  	<limit effort="1000.0" lower="-6.28" upper="6.28" velocity="0.2"/>
+  <joint name="head_joint" type="fixed">
   	<origin rpy="0 0 0" xyz="0 0 0.05"/>
   	<parent link="neck_link"/>
@@ -169,5 +168,5 @@
   <link name="camera_link">
 	    <collision>
-	      <origin xyz="0 0 0.025" rpy="0 0 0"/>
+	      <origin xyz="0 0 0.005" rpy="0 0 0"/>
 	      <geometry>
 		<box size="0.05 0.05 0.01"/>
@@ -195,3 +194,13 @@
 	    <child link="camera_link"/>
 	 </joint>
+<transmission name="neck_joint_trans">
+	<type>transmission_interface/SimpleTransmission</type>
+	<joint name="neck_joint">
+		<hardwareInterface>hardware_interface/EffortJointInterface</hardwareInterface>
+	</joint>
+	<actuator name="motor1">
+		<hardwareInterface>hardware_interface/EffortJointInterface</hardwareInterface>
+		<mechanicalInterface>1</mechanicalInterface>
+	</actuator>
+</transmission>
 </robot>
